Commit message: Update diffbot system to work better

File: description/ros2_control/diffbot.ros2_control.xacro (robot description, xacro)
@@ -2,19 +2,19 @@
 <robot xmlns:xacro="http://www.ros.org/wiki/xacro">
   <xacro:macro name="diffbot_ros2_control" params="name prefix">
-    <ros2_control name="${name}" type="system">
+    <ros2_control name="diffdrive" type="system">
       <hardware>
         <plugin>diffdrive_mini_ocebot/DiffBotSystemHardware</plugin>
-        <param name="left_wheel_name">left_front</param>
-        <param name="right_wheel_name">right_rear</param>
+        <param name="left_wheel_name">left_wheel_joint</param>
+        <param name="right_wheel_name">right_wheel_joint</param>
         <param name="left_wheel_pin">25</param>
         <param name="right_wheel_pin">10</param>
         <param name="enc_counts_per_rev">3640</param>
       </hardware>
-      <joint name="${prefix}left_wheel_joint">
+      <joint name="left_wheel_joint">
         <command_interface name="velocity"/>
         <state_interface name="position"/>
         <state_interface name="velocity"/>
       </joint>
-      <joint name="${prefix}right_wheel_joint">
+      <joint name="right_wheel_joint">
         <command_interface name="velocity"/>
         <state_interface name="position"/>
